File: Version_B/Bottom_Board/Hardware_Filter.kicad_sch (KiCad schematic)
At the start: 38 parts, among them U1 LM324, U2 LM324

Commit message: added flash folder and adjusted GUI
Other:
- company: (none) -> Secured Solutions Group
- title: Current Monitoring System -> Current Monitoring System (Bottom Board)
Changed lines of the file:
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@@
 	(paper "A4")
 	(title_block
-		(title "Current Monitoring System")
-		(date "2024-02-23")
+		(title "Current Monitoring System (Bottom Board)")
+		(date "2024-03-05")
 		(rev "C1.04")
+		(company "Secured Solutions Group")
+		(comment 1 "David Nguyen")
+		(comment 2 "david@securedsolutionsgroup.com")
+		(comment 3 "(909)-896-1654")
 	)
 	(junction

Commit message: minor fixe
Parts:
- RV21, RV7: value 20K -> 20K POT
- U1, U2: value LM324 -> LM324DR
Changed lines of the file:
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@@
 			)
 		)
-		(property "Value" "LM324"
+		(property "Value" " LM324DR"
 			(at 99.06 68.58 0)
 			(effects
@@
 			)
 		)
-		(property "Value" "LM324"
+		(property "Value" " LM324DR"
 			(at 248.285 76.2 0)
 			(effects
@@
 			)
 		)
-		(property "Value" "LM324"
+		(property "Value" " LM324DR"
 			(at 90.805 153.035 0)
 			(effects
@@
 			)
 		)
-		(property "Value" "20K"
+		(property "Value" "20K POT"
 			(at 211.455 100.965 0)
 			(effects
@@
 			)
 		)
-		(property "Value" "LM324"
+		(property "Value" " LM324DR"
 			(at 60.96 66.675 0)
 			(effects
@@
 			)
 		)
-		(property "Value" "LM324"
+		(property "Value" " LM324DR"
 			(at 131.445 66.04 0)
 			(effects
@@
 			)
 		)
-		(property "Value" "LM324"
+		(property "Value" " LM324DR"
 			(at 180.975 74.295 0)
 			(effects
@@
 			)
 		)
-		(property "Value" "LM324"
+		(property "Value" " LM324DR"
 			(at 152.4 153.67 0)
 			(effects
@@
 			)
 		)
-		(property "Value" "LM324"
+		(property "Value" " LM324DR"
 			(at 46.99 160.655 0)
 			(effects
@@
 			)
 		)
-		(property "Value" "LM324"
+		(property "Value" " LM324DR"
 			(at 123.825 154.94 0)
 			(effects
@@
 			)
 		)
-		(property "Value" "20K"
+		(property "Value" "20K POT"
 			(at 85.09 91.44 90)
 			(effects
@@
 			)
 		)
-		(property "Value" "LM324"
+		(property "Value" " LM324DR"
 			(at 58.42 160.02 0)
 			(effects

Commit message: switched B and C directories
Parts:
- removed R11: 1M, Resistor_SMD:R_0603_1608Metric, symbol Device:R_US
- removed unit 1 of U2
- removed unit 4 of U2
- removed unit 3 of U2
- D1: value 1N4148WS -> 1N914; footprint bot_lib:Diode_1N4148WS -> Diode_SMD:D_0603_1608Metric
- RV21, RV7: value 20K POT -> 20K; footprint bot_lib:Potentiometer_Bourns_3386P_Vertical -> Potentiometer_THT:Potentiometer_Bourns_3386P_Vertical
- U1, U2: value LM324DR -> LM324
Connections:
- net at R7.1, R9.2, U1.6 (-): now also RV7.2
- net at C11.1, R3.1, U1.9 (-): no longer R4.1, R5.1
- net 2x_OUTPUT: now reaches R25.1, R26.2
- net +5VD renamed +5V
- net AN0 renamed 4x_OUTPUT
- new net: R4.1, R5.1
Other:
- note removed: "Unused OPAMPS"
- company: Secured Solutions Group -> (none)
- title: Current Monitoring System (Bottom Board) -> (none)
- moved on the sheet: C11, C2, C3, C4, C7, D1, R1, R11, R13, R14, R15, R16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

Commit message: updated board b
Changed lines of the file:
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@@
   )
   (symbol (lib_id "Device:R_US") (at 81.915 143.51 270) (unit 1)
-    (in_bom yes) (on_board yes) (dnp no) (fields_autoplaced)
+    (in_bom yes) (on_board yes) (dnp no)
     (property "Reference" "R23" (at 81.915 139.065 90)
       (effects (font (size 1.27 1.27)))
     )
-    (property "Value" "1M" (at 81.915 141.605 90)
+    (property "Value" "1M" (at 82.55 140.97 90)
       (effects (font (size 1.27 1.27)))
     )

Commit message: adjusted hardware values
Parts:
- added R11: 1M, Resistor_SMD:R_0603_1608Metric, symbol Device:R_US
Connections:
- net 2x_OUTPUT: now also R26.1, R27.2; no longer R25.1, R26.2
- net 4x_OUTPUT: now also R25.1, R26.2; no longer R26.1, R27.2
- net at R7.1, R9.2, U1.6 (-): now also R11.1; no longer RV7.2
- net at C11.1, R3.1, U1.9 (-): now also R4.1, R5.1
- new net: R11.2, RV7.2
Other:
- moved on the sheet: R4

Commit message: updated simulation circuit and finalized hardware design?
Changed lines of the file:
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@@
   (junction (at 151.13 49.53) (diameter 0) (color 0 0 0 0)
   )
-  (junction (at 86.995 49.53) (diameter 0) (color 0 0 0 0)
+  (junction (at 86.36 49.53) (diameter 0) (color 0 0 0 0)
   )
   (junction (at 76.2 116.205) (diameter 0) (color 0 0 0 0)
@@
     (stroke (width 0) (type default))
   )
-  (wire (pts (xy 85.725 49.53) (xy 86.995 49.53))
+  (wire (pts (xy 85.725 49.53) (xy 86.36 49.53))
     (stroke (width 0) (type default))
   )
@@
     (stroke (width 0) (type default))
   )
-  (wire (pts (xy 86.995 52.705) (xy 86.995 49.53))
+  (wire (pts (xy 86.36 52.705) (xy 86.36 49.53))
     (stroke (width 0) (type default))
   )
@@
     (stroke (width 0) (type default))
   )
-  (wire (pts (xy 74.295 52.705) (xy 86.995 52.705))
+  (wire (pts (xy 74.295 52.705) (xy 86.36 52.705))
     (stroke (width 0) (type default))
   )
@@
     (stroke (width 0) (type default))
   )
-  (wire (pts (xy 86.995 49.53) (xy 88.9 49.53))
+  (wire (pts (xy 86.36 49.53) (xy 88.9 49.53))
     (stroke (width 0) (type default))
   )
