File: Version_B/Bottom_Board/Bottom_Board.kicad_pcb (KiCad board)
At the start: 2 copper layers, 74.8 x 84.5 mm, 52 parts, among them J1 Conn_02x03_Top_Bottom, J2 Conn_02x03_Top_Bottom, J3 Conn_01x02_Pin, J5 DIN-5, J6 Conn_01x02_Pin, J7 Conn_01x02_Pin, J8 Screw_Terminal_01x04, J9 Screw_Terminal_01x04, SW2 SW_DIP_x04, U1 LM324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

Commit message: 90 degree terminal block added
Parts:
- moved J5 1.50 mm to (168.1, 126.8)
- moved J9 0.94 mm to (166.1, 106.9)
Routing:
- net AN1: track 240.5 -> 267.3 mm, vias 2 -> 6
- net -5V: track 91.6 -> 92.4 mm
Other:
- board text added: "VC1.03"
- board text removed: "E- GND"
- board text removed: "VC1.02"
