File: Version_B/Bottom_Board/Bottom_Board.kicad_sch (KiCad schematic)
At the start: 13 parts, among them J1 Conn_02x03_Top_Bottom, J2 Conn_02x03_Top_Bottom, J3 Conn_01x02_Pin, J5 DIN-5, J6 Conn_01x02_Pin, J7 Conn_01x02_Pin, J8 Screw_Terminal_01x04, J9 Screw_Terminal_01x04, SW2 SW_DIP_x04

Commit message: 90 degree terminal block added
Other:
- company: (none) -> Secured Solutions Group
- title: (none) -> Monitoring System (Bottom Board)
Changed lines of the file:
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@@
 (kicad_sch (version 20230121) (generator eeschema)
   (paper "A4")
+  (title_block
+    (title "Monitoring System (Bottom Board)")
+    (date "2024-02-24")
+    (rev "C1.03")
+    (company "Secured Solutions Group")
+  )
   (junction (at 81.915 120.65) (diameter 0) (color 0 0 0 0)
   )
