File: Version_B/Top_Board/Top_Board.kicad_pcb (KiCad board)
At the start: 2 copper layers, 78.7 x 31 mm, 5 parts, among them J1 90_Deg_Conn, J2 90_Deg_Conn, U1 T-Display-S3

Commit message: updated jlpcb format
Other:
- board text added: "VerC1.05"
- board text removed: "VerC1.04"
